File: wpcpowermon.kicad_sch (KiCad schematic)
At the start: 14 parts, among them J1 Screw_Terminal_01x02, U1 74HC245, U2 6808, U3 74HC245, U4 74HC245, U5 Pico, U6 MAX485E

Commit message: First PCB draft
Parts:
- removed U1: 74HC245, Package_DIP:DIP-20_W7.62mm_LongPads, symbol 74xx:74HC245
- removed U2: 6808, Package_DIP:DIP-40_W15.24mm, symbol CPU_NXP_6800:MC68A00
- added J1001: Conn_02x17_Odd_Even, Connector_PinHeader_2.54mm:PinHeader_2x17_P2.54mm_Vertical, symbol Connector_Generic:Conn_02x17_Odd_Even
Connections:
- net D0: now also U4.18 (B0)
- net D1: now also U4.17 (B1)
- net D2: now also U4.16 (B2)
- net D3: now also U4.15 (B3)
- net D4: now also U4.14 (B4)
- net D5: now also U4.13 (B5)
- net D6: now also U4.12 (B6)
- net D7: now also U4.11 (B7)
- net GND: now also J1001.14 (Pin_14), J1001.16 (Pin_16), J1001.18 (Pin_18), J1001.20 (Pin_20), J1001.22 (Pin_22), J1001.24 (Pin_24), J1001.26 (Pin_26), J1001.28 (Pin_28), J1001.30 (Pin_30)
- net /ZEROCROSS: now reaches U3.11 (B7)
- net /ZEROCROSS: now also U5.20 (GPIO15)
- net /LAMP ROW: now reaches U3.12 (B6)
- net /LAMP ROW: now also U5.19 (GPIO14)
- net /LAMP COL: now reaches U3.13 (B5)
- net /LAMP COL: now also U5.17 (GPIO13)
- net /SOL2: now reaches U3.14 (B4)
- net /SOL2: now also U5.16 (GPIO12)
- net /TRIACS: now reaches U3.18 (B0)
- net /TRIACS: now also U5.11 (GPIO8)
- net at U3.2 (A0): now also J1001.13 (Pin_13)
- net at U3.3 (A1): now also J1001.12 (Pin_12)
- net at U3.4 (A2): now also J1001.11 (Pin_11)
- net at U3.5 (A3): now also J1001.10 (Pin_10)
- net at U3.6 (A4): now also J1001.9 (Pin_9)
- net at U3.7 (A5): now also J1001.8 (Pin_8)
- net at U3.8 (A6): now also J1001.7 (Pin_7)
- net at U3.9 (A7): now also J1001.34 (Pin_34)
- net at U4.2 (A0): now also J1001.29 (Pin_29)
- net at U4.3 (A1): now also J1001.27 (Pin_27)
- net at U4.4 (A2): now also J1001.25 (Pin_25)
- net at U4.5 (A3): now also J1001.23 (Pin_23)
- net at U4.6 (A4): now also J1001.21 (Pin_21)
- net at U4.7 (A5): now also J1001.19 (Pin_19)
- net at U4.8 (A6): now also J1001.17 (Pin_17)
- net at U4.9 (A7): now also J1001.15 (Pin_15)
- net A10 renamed /SOL3
- net /SOL3: now also U3.16 (B2); no longer U4.16 (B2)
- net A11 renamed /SOL4
- net /SOL4: now also U3.15 (B3); no longer U4.15 (B3)
- removed net A12: U4.14 (B4), U5.16 (GPIO12)
- removed net A13: U4.13 (B5), U5.17 (GPIO13)
- removed net A14: U4.12 (B6), U5.19 (GPIO14)
- removed net A15: U4.11 (B7), U5.20 (GPIO15)
- removed net A8: U4.18 (B0), U5.11 (GPIO8)
- net A9 renamed /SOL1
- net /SOL1: now also U3.17 (B1); no longer U4.17 (B1)
- net E: no longer names the net of U5.32 (GPIO27_ADC1)
- net E: no longer U3.15 (B3)
- net R/W: no longer names the net of U5.29 (GPIO22)
- net R/W: no longer U3.16 (B2)
- net VMA: no longer names the net of U5.31 (GPIO26_ADC0)
- net VMA: no longer U3.17 (B1)
- no-connect marks 17 -> 12

Commit message: Version 0.1
Parts:
- removed J1: Screw_Terminal_01x02, TerminalBlock_4Ucon:TerminalBlock_4Ucon_1x02_P3.50mm_Horizontal, symbol Connector:Screw_Terminal_01x02
- added J1: Screw_Terminal_01x04, TerminalBlock_4Ucon:TerminalBlock_4Ucon_1x04_P3.50mm_Horizontal, symbol Connector:Screw_Terminal_01x04
- added J2, J3: LED, Connector_Molex:Molex_SL_171971-0004_1x04_P2.54mm_Vertical, symbol Connector:Conn_01x04_Male
- added J4: Screw_Terminal_01x02, TerminalBlock_4Ucon:TerminalBlock_4Ucon_1x02_P3.50mm_Horizontal, symbol Connector:Screw_Terminal_01x02
Connections:
- net +3V3: no longer C3.1
- net +5V: now also C3.1, U6.8 (VCC), J1.1 (Pin_1), J2.1 (Pin_1), J3.1 (Pin_1), J4.1 (Pin_1)
- net GND: now also U6.5 (GND), J1.4 (Pin_4), J2.4 (Pin_4), J3.4 (Pin_4), J4.2 (Pin_2)
- net at R1.1, U6.6 (A): now also J1.2 (Pin_2)
- net at JP1.1, U6.7 (B): now also J1.3 (Pin_3)
- net at U5.26 (GPIO20): now also J3.3 (Pin_3)
- net at U5.27 (GPIO21): now also J3.2 (Pin_2)
- net at U5.32 (GPIO27_ADC1): now also J2.3 (Pin_3)
- net at U5.34 (GPIO28_ADC2): now also J2.2 (Pin_2)
Other:
- moved on the sheet: C1, C2, C3, D1, J1001, JP1, R1, R2, U3, U4, U5, U6

Commit message: v 0.2
Parts:
- removed J1: Screw_Terminal_01x04, TerminalBlock_4Ucon:TerminalBlock_4Ucon_1x04_P3.50mm_Horizontal, symbol Connector:Screw_Terminal_01x04
- removed J2, J3: LED, Connector_Molex:Molex_SL_171971-0004_1x04_P2.54mm_Vertical, symbol Connector:Conn_01x04_Male
- removed JP1: Jumper, Connector_PinHeader_2.54mm:PinHeader_1x02_P2.54mm_Vertical, symbol Device:Jumper
- removed R1: R, Resistor_THT:R_Axial_DIN0204_L3.6mm_D1.6mm_P5.08mm_Horizontal, symbol Device:R
- removed U6: MAX485E, Package_DIP:DIP-8_W7.62mm_LongPads, symbol Interface_UART:MAX485E
- J1001: value Conn_02x17_Odd_Even -> WPC Bus
- J4: value Screw_Terminal_01x02 -> 5V
- R2: value R -> 470R
- U3, U4: value 74HC245 -> 74LVC245
Connections:
- net +5V: now also D1.2 (A)
- net io/IO5: now reaches U5.27 (GPIO21)
- net io/IO6: now reaches U5.26 (GPIO20)
- net io/RX: now reaches U5.22 (GPIO17)
- net io/IO8: now reaches U5.24 (GPIO18)
- net io/TX: now reaches U5.21 (GPIO16)
- net io/IO1: now reaches U5.34 (GPIO28_ADC2)
- net io/IO2: now reaches U5.32 (GPIO27_ADC1)
- net io/IO7: now reaches U5.25 (GPIO19)
- net io/IO7: no longer D1.2 (A)
- net io/IO4: now reaches U5.29 (GPIO22)
- net io/IO3: now reaches U5.31 (GPIO26_ADC0)
- no-connect marks 12 -> 6
Other:
- added sheet io (io.kicad_sch)
- moved on the sheet: U3
